File: kicad/synthboard.kicad_pcb (KiCad board)
At the start: 2 copper layers, 47 parts, among them J1 Connection to Upper Module/FP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, J2 Connection to Lower Module, J3 Modular Inputs, SW1 SW_Push, SW10 SW_Push, SW11 SW_Push, SW12 SW_Push, SW2 SW_Push, SW3 SW_Push, SW4 SW_Push, SW5 SW_Push, SW6 SW_Push, SW7 SW_Push, SW8 SW_Push, SW9 SW_Push, U1 74HC165, U2 74HC165

Commit message: first draft PCB design done
Will look for errors with fresh eyes later.
Parts:
- J1: value Connection to Upper Module/FPGA -> Connect to Upper Module/FPGA
- J2: value Connection to Lower Module -> Connect to Lower Module
- R10, R11, R12, R13, R2, R3, R4, R5, R6, R7, R8, R9: moved to B.Cu
- moved R13 183.4 mm to (265.0, 129.3), turned to -90 degrees
- moved R12 165.3 mm to (247.9, 132.4), turned to 180 degrees
- moved C4 158.2 mm to (76.9, 118.1), turned to 90 degrees
- moved R11 144.7 mm to (227.4, 132.5), turned to 180 degrees
- moved R10 122.1 mm to (204.0, 129.5), turned to -90 degrees
- moved C3 116.4 mm to (137.9, 118.1), turned to 90 degrees
- moved C1 113.8 mm to (259.8, 118.0), turned to 90 degrees
- moved R9 111.9 mm to (186.9, 132.4), turned to 180 degrees
- moved C2 97.6 mm to (198.8, 118.1), turned to 90 degrees
- moved R8 92.4 mm to (166.4, 131.1), turned to 180 degrees
- moved R7 73.0 mm to (146.1, 131.0), turned to 180 degrees
- moved R6 54.2 mm to (125.8, 131.1), turned to 180 degrees
- moved R5 46.6 mm to (99.3, 131.1)
- moved R2 45.4 mm to (44.9, 132.5), turned to 180 degrees
- moved R3 36.5 mm to (65.0, 132.4), turned to 180 degrees
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Routing:
- net GND: track 3.92 -> 83.2 mm, vias 0 -> 113
- net +5V: track 230.8 -> 275.4 mm
- net +3.3V: track 3.94 -> 11.5 mm, vias 0 -> 10
- net Shift Reg Latch: track 251.0 -> 257.4 mm
- net Shift Reg Clock: track 154.7 -> 151.9 mm
- net SW3: track 28.1 -> 30.9 mm
- net SW6: track 33.0 -> 35.7 mm
- net SW5: track 12.2 -> 14.9 mm
- net SW7: track 53.8 -> 56.5 mm
- net SW4: track 8.52 -> 11.2 mm
- net SW1: track 69.7 -> 72.4 mm
- net SW2: track 48.9 -> 51.3 mm
- net SW11: track 36.2 -> 38.6 mm
- net SW8: track 74.7 -> 77.0 mm
- net SW10: track 14.2 -> 16.5 mm
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- added copper zone on In1.Cu, net +3.3V
- added copper zone on In2.Cu, net GND
Other:
- board outline added: 243.9 x 39.9 mm
- copper layers 2 -> 4
- board text added: "+3.3V"
- board text added: "GND"
- board text added: "MOD 1"
- board text added: "MOD 2"
- board text added: "MOD 3"
- board text added: "MOD 4"
