File: kicad/4/synthboard.kicad_pcb (KiCad board)
At the start: 4 copper layers, 243.9 x 39.9 mm, 47 parts, among them J1 Connect to Upper Module/FPGA, J2 Connect to Lower Module, J3 Modular Inputs, SW1 SW_Push, SW10 SW_Push, SW11 SW_Push, SW12 SW_Push, SW2 SW_Push, SW3 SW_Push, SW4 SW_Push, SW5 SW_Push, SW6 SW_Push, SW7 SW_Push, SW8 SW_Push, SW9 SW_Push, U1 74HC165, U2 74HC165

Commit message: Added 2 layer board
4 layer board has been separated into separate folder.
The 2 layer board passes DRC.
Need to potentially revise schematic. I think the shift registers may not be talking to each other with just one communicating with the data in/out pins on the board.
Routing:
- net Shift Reg Latch: track 257.4 -> 193.1 mm
- net Shift Reg Clock: track 151.9 -> 190.4 mm
- net SW5: track 14.9 -> 20.2 mm
- net (no net): track 1.70 -> 0.00 mm
- net Shift Data In: track 208.0 -> 206.7 mm
- net SW6: track 35.7 -> 37.0 mm
- net SW12: track 60.4 -> 61.7 mm
- net +3.3V: track 11.5 -> 10.2 mm, vias 10 -> 8
- net GND: track 83.2 -> 84.4 mm, vias 113 -> 107
- net SW7: track 56.5 -> 57.1 mm
- net SW4: track 11.2 -> 11.7 mm
- net Shift Data Out: track 181.1 -> 181.7 mm
