File: kicad/2_layer_zones/synthboard.kicad_pcb (KiCad board)
At the start: 2 copper layers, 243.9 x 39.9 mm, 47 parts, among them J1 Connect to Upper Module/FPGA, J2 Connect to Lower Module, J3 Modular Inputs, SW1 SW_Push, SW10 SW_Push, SW11 SW_Push, SW12 SW_Push, SW2 SW_Push, SW3 SW_Push, SW4 SW_Push, SW5 SW_Push, SW6 SW_Push, SW7 SW_Push, SW8 SW_Push, SW9 SW_Push, U1 74HC165, U2 74HC165

Commit message: 2 layer board rev 1 tentatively finished
Hoping for a design review
Parts:
- added H1: MountingHole, MountingHole:MountingHole_3.2mm_M3, F.Cu at (32.4, 103.5)
- added H2: MountingHole, MountingHole:MountingHole_3.2mm_M3, F.Cu at (268.8, 103.5)
- added H3: MountingHole, MountingHole:MountingHole_3.2mm_M3, F.Cu at (32.4, 152.1)
- added H4: MountingHole, MountingHole:MountingHole_3.2mm_M3, F.Cu at (268.9, 152.1)
- J1: value Connect to Upper Module/FPGA -> Connection to Upper Module/FPGA
- J2: value Connect to Lower Module -> Connection to Lower Module
Connections:
- J3 pad 3: Modular Input 1 -> Modular Input 4
- J3 pad 4: Modular Input 2 -> Modular Input 3
- J3 pad 5: Modular Input 3 -> Modular Input 2
- J3 pad 6: Modular Input 4 -> Modular Input 1
- U1 pad 9: Shift Data Out -> Shift Data In
- U2 pad 10: Shift Data In -> Shift Data Out
Routing:
- net Shift Data In: track 209.0 -> 97.5 mm
- net +3.3V: track 46.0 -> 150.9 mm, vias 4 -> 3
- net Shift Data Out: track 181.1 -> 81.6 mm
- net Modular Input 4: track 60.0 -> 69.0 mm, vias 1 -> 2
- net +5V: track 274.4 -> 282.5 mm
- net SW5: track 14.9 -> 21.5 mm
- net Modular Input 1: track 70.9 -> 65.2 mm, vias 1 -> 2
- net Modular Input 3: track 63.4 -> 67.7 mm, vias 1 -> 2
- net Shift Reg Clock: track 257.6 -> 259.1 mm, vias 2 -> 0
- net SW9: track 16.2 -> 15.1 mm
- net SW6: track 36.6 -> 37.6 mm
- net Shift Reg Latch: track 257.6 -> 258.4 mm
- net Modular Input 2: track 66.9 -> 66.5 mm, vias 0 -> 2
Other:
- board size 243.9 x 39.9 mm -> 243.9 x 55.9 mm
