File: kicad/2_layer_zones/synthboard.kicad_sch (KiCad schematic)
At the start: 47 parts, among them J1 Connection to Upper Module/FP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, J2 Connection to Lower Module, J3 Modular Inputs, SW1 SW_Push, SW10 SW_Push, SW11 SW_Push, SW12 SW_Push, SW2 SW_Push, SW3 SW_Push, SW4 SW_Push, SW5 SW_Push, SW6 SW_Push, SW7 SW_Push, SW8 SW_Push, SW9 SW_Push, U1 74HC165, U2 74HC165

Commit message: 2 layer board rev 1 tentatively finished
Hoping for a design review
Parts:
- added H1, H2, H3, H4: MountingHole, MountingHole:MountingHole_3.2mm_M3, symbol Mechanical:MountingHole
Connections:
- net Modular Input 1: now also J3.6 (Pin_6); no longer J3.3 (Pin_3)
- net Modular Input 2: now also J3.5 (Pin_5); no longer J3.4 (Pin_4)
- net Modular Input 3: now also J3.4 (Pin_4); no longer J3.5 (Pin_5)
- net Modular Input 4: now also J3.3 (Pin_3); no longer J3.6 (Pin_6)
- net Shift Data In: now also U1.9 (Q7); no longer U2.10 (DS)
- net Shift Data Out: now also U2.10 (DS); no longer U1.9 (Q7)
Other:
- note added: "Screw/Mounting Holes"
- moved on the sheet: U1, U2
